File: KiCad/UniDCBuckHW.kicad_pcb (KiCad board)
At the start: 2 copper layers, 66 x 32 mm, 36 parts, among them J1 IN, J2 12V, J3 i2c, J4 LOAD, J5 PROG, Q1 IRLR8726PBF, U1 LM2940-12V, U2 MCP1703-5V, U3 IR2101, U4 ATTINY85-20SU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

Commit message: Final Vq PCB
Parts:
- added C16: 10uf, Capacitors_SMD:C_0603, F.Cu at (220.4, 110.3)
- added D4: LED, LEDs:LED_0805, F.Cu at (197.1, 138.7)
- added R5: 2K, Resistors_SMD:R_0603, F.Cu at (197.8, 135.7)
Routing:
- net GND: track 230.0 -> 257.4 mm, vias 62 -> 63
- net Net-(C6-Pad1): track 55.7 -> 68.1 mm, vias 2 -> 6
- net Net-(D4-Pad2): track 0.00 -> 3.42 mm
- net +12V: track 88.0 -> 89.7 mm
- net +5V: track 83.8 -> 84.6 mm
- added copper zone on B.Cu, net Net-(C6-Pad1)
Other:
- board text added: "PWR"
