File: KiCad/UniDCBuckHW.sch (KiCad schematic (older format))
At the start: 34 parts, among them J1 IN, J2 12V, J3 i2c, J4 LOAD, J5 PROG, Q1 IRLR8726PBF, U1 LM2940-12V, U2 MCP1703-5V, U3 IR2101, U4 ATTINY85-20SU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

Commit message: Final Vq PCB
Parts:
- added C16: 10uf, Capacitors_SMD:C_0603, symbol C
- added D4: LED, LEDs:LED_0805, symbol LED
- added R5: 2K, Resistors_SMD:R_0603, symbol R
Connections:
- net +12V: now also R5.2
- net +5V: now also C16.2
- net GND: now also C16.1, D4.1 (K)
- new net: D4.2 (A), R5.1
Changed lines of the file:
@@
 	7500 3750 8350 3750
 $Comp
-L GND #PWR17
+L GND #PWR19
 U 1 1 5B64CE60
 P 7350 3850
-F 0 "#PWR17" H 7350 3600 50  0001 C CNN
+F 0 "#PWR19" H 7350 3600 50  0001 C CNN
 F 1 "GND" H 7350 3700 50  0000 C CNN
 F 2 "" H 7350 3850 50  0001 C CNN
@@
 Connection ~ 5500 4300
 $Comp
-L GND #PWR16
+L GND #PWR18
 U 1 1 5B64D0A8
 P 5500 4400
-F 0 "#PWR16" H 5500 4150 50  0001 C CNN
+F 0 "#PWR18" H 5500 4150 50  0001 C CNN
 F 1 "GND" H 5500 4250 50  0000 C CNN
 F 2 "" H 5500 4400 50  0001 C CNN
@@
 Connection ~ 6500 3150
 $Comp
-L GND #PWR13
+L GND #PWR15
 U 1 1 5B64DE14
 P 4950 3800
-F 0 "#PWR13" H 4950 3550 50  0001 C CNN
+F 0 "#PWR15" H 4950 3550 50  0001 C CNN
 F 1 "GND" H 4950 3650 50  0000 C CNN
 F 2 "" H 4950 3800 50  0001 C CNN
@@
 $EndComp
 $Comp
-L GND #PWR18
+L GND #PWR20
 U 1 1 5B64DF9C
 P 8250 5500
-F 0 "#PWR18" H 8250 5250 50  0001 C CNN
+F 0 "#PWR20" H 8250 5250 50  0001 C CNN
 F 1 "GND" H 8250 5350 50  0000 C CNN
 F 2 "" H 8250 5500 50  0001 C CNN
@@
 U 1 1 5B64E541
 P 8000 5250
-F 0 "C11" H 7900 5350 50  0000 L CNN
+F 0 "C11" H 7850 5350 50  0000 L CNN
 F 1 "100n" H 7800 5150 50  0000 L CNN
 F 2 "Capacitors_SMD:C_0603" H 8038 5100 50  0001 C CNN
@@
 U 1 1 5B64E5A7
 P 8400 5250
-F 0 "C13" H 8300 5350 50  0000 L CNN
+F 0 "C13" H 8250 5350 50  0000 L CNN
 F 1 "22uf" H 8200 5150 50  0000 L CNN
 F 2 "Capacitors_SMD:C_0805" H 8438 5100 50  0001 C CNN
@@
 $EndComp
 $Comp
-L GND #PWR14
+L GND #PWR16
 U 1 1 5B64EB5B
 P 5150 4400
-F 0 "#PWR14" H 5150 4150 50  0001 C CNN
+F 0 "#PWR16" H 5150 4150 50  0001 C CNN
 F 1 "GND" H 5150 4250 50  0000 C CNN
 F 2 "" H 5150 4400 50  0001 C CNN
@@
 Vsense
 $Comp
-L GND #PWR12
+L GND #PWR14
 U 1 1 5B65D7CD
 P 4400 5900
-F 0 "#PWR12" H 4400 5650 50  0001 C CNN
+F 0 "#PWR14" H 4400 5650 50  0001 C CNN
 F 1 "GND" H 4400 5750 50  0000 C CNN
 F 2 "" H 4400 5900 50  0001 C CNN
@@
 $EndComp
 $Comp
-L GND #PWR21
+L GND #PWR23
 U 1 1 5B65E07C
 P 9550 5100
-F 0 "#PWR21" H 9550 4850 50  0001 C CNN
+F 0 "#PWR23" H 9550 4850 50  0001 C CNN
 F 1 "GND" H 9550 4950 50  0000 C CNN
 F 2 "" H 9550 5100 50  0001 C CNN
@@
 U 1 1 5B65E252
 P 10150 4850
-F 0 "C15" H 10050 4950 50  0000 L CNN
+F 0 "C15" H 10000 4950 50  0000 L CNN
 F 1 "1n" H 10000 4750 50  0000 L CNN
 F 2 "Capacitors_SMD:C_0603" H 10188 4700 50  0001 C CNN
@@
 	9950 4700 10150 4700
 $Comp
-L +5V #PWR20
+L +5V #PWR22
 U 1 1 5B65E6CB
 P 9550 3750
-F 0 "#PWR20" H 9550 3600 50  0001 C CNN
+F 0 "#PWR22" H 9550 3600 50  0001 C CNN
 F 1 "+5V" H 9550 3890 50  0000 C CNN
 F 2 "" H 9550 3750 50  0001 C CNN
@@
 U 1 1 5B65E87A
 P 10050 3950
-F 0 "C14" H 9950 4050 50  0000 L CNN
+F 0 "C14" H 9900 4050 50  0000 L CNN
 F 1 "100n" H 9850 3850 50  0000 L CNN
 F 2 "Capacitors_SMD:C_0603" H 10088 3800 50  0001 C CNN
@@
 Connection ~ 9550 3800
 $Comp
-L GND #PWR22
+L GND #PWR24
 U 1 1 5B65EBE3
 P 10050 4100
-F 0 "#PWR22" H 10050 3850 50  0001 C CNN
+F 0 "#PWR24" H 10050 3850 50  0001 C CNN
 F 1 "GND" H 10050 3950 50  0000 C CNN
 F 2 "" H 10050 4100 50  0001 C CNN
@@
 Connection ~ 3450 4850
 $Comp
-L GND #PWR7
+L GND #PWR9
 U 1 1 5B66149A
 P 3450 4850
-F 0 "#PWR7" H 3450 4600 50  0001 C CNN
+F 0 "#PWR9" H 3450 4600 50  0001 C CNN
 F 1 "GND" H 3450 4700 50  0000 C CNN
 F 2 "" H 3450 4850 50  0001 C CNN
@@
 $EndComp
 $Comp
-L +5V #PWR19
+L +5V #PWR21
 U 1 1 5B6617BD
 P 8400 5000
-F 0 "#PWR19" H 8400 4850 50  0001 C CNN
+F 0 "#PWR21" H 8400 4850 50  0001 C CNN
 F 1 "+5V" H 8400 5140 50  0000 C CNN
 F 2 "" H 8400 5000 50  0001 C CNN
@@
 Connection ~ 8400 5000
 $Comp
-L +5V #PWR11
+L +5V #PWR13
 U 1 1 5B661860
 P 3950 4550
-F 0 "#PWR11" H 3950 4400 50  0001 C CNN
+F 0 "#PWR13" H 3950 4400 50  0001 C CNN
 F 1 "+5V" H 3950 4690 50  0000 C CNN
 F 2 "" H 3950 4550 50  0001 C CNN
@@
 $EndComp
 $Comp
-L +12V #PWR10
+L +12V #PWR12
 U 1 1 5B662124
 P 3950 3850
-F 0 "#PWR10" H 3950 3700 50  0001 C CNN
+F 0 "#PWR12" H 3950 3700 50  0001 C CNN
 F 1 "+12V" H 3950 3990 50  0000 C CNN
 F 2 "" H 3950 3850 50  0001 C CNN
@@
 Wire Wire Line
 	2900 4150 4350 4150
-Wire Wire Line
-	2900 3850 2900 3650
 Connection ~ 4950 3150
 Connection ~ 2900 3850
 Connection ~ 3450 4150
 $Comp
-L GND #PWR6
+L GND #PWR8
 U 1 1 5B6635F3
 P 3450 4150
-F 0 "#PWR6" H 3450 3900 50  0001 C CNN
+F 0 "#PWR8" H 3450 3900 50  0001 C CNN
 F 1 "GND" H 3450 4000 50  0000 C CNN
 F 2 "" H 3450 4150 50  0001 C CNN
@@
 Connection ~ 3950 3850
 $Comp
-L +12V #PWR15
+L +12V #PWR17
 U 1 1 5B6645D9
 P 5500 3300
-F 0 "#PWR15" H 5500 3150 50  0001 C CNN
+F 0 "#PWR17" H 5500 3150 50  0001 C CNN
 F 1 "+12V" H 5500 3440 50  0000 C CNN
 F 2 "" H 5500 3300 50  0001 C CNN
@@
 Connection ~ 5500 3300
 $Comp
-L +12V #PWR5
+L +12V #PWR7
 U 1 1 5B664929
 P 2900 4550
-F 0 "#PWR5" H 2900 4400 50  0001 C CNN
+F 0 "#PWR7" H 2900 4400 50  0001 C CNN
 F 1 "+12V" H 2900 4690 50  0000 C CNN
 F 2 "" H 2900 4550 50  0001 C CNN
@@
 Connection ~ 2900 3150
 $Comp
-L GND #PWR1
+L GND #PWR2
 U 1 1 5B666BBE
 P 2350 3250
-F 0 "#PWR1" H 2350 3000 50  0001 C CNN
+F 0 "#PWR2" H 2350 3000 50  0001 C CNN
 F 1 "GND" H 2350 3100 50  0000 C CNN
 F 2 "" H 2350 3250 50  0001 C CNN
@@
 $EndComp
 $Comp
-L +12V #PWR2
+L +12V #PWR3
 U 1 1 5B6678CE
 P 2350 4300
-F 0 "#PWR2" H 2350 4150 50  0001 C CNN
+F 0 "#PWR3" H 2350 4150 50  0001 C CNN
 F 1 "+12V" H 2350 4440 50  0000 C CNN
 F 2 "" H 2350 4300 50  0001 C CNN
@@
 $EndComp
 $Comp
-L GND #PWR3
+L GND #PWR4
 U 1 1 5B667A19
 P 2350 4400
-F 0 "#PWR3" H 2350 4150 50  0001 C CNN
+F 0 "#PWR4" H 2350 4150 50  0001 C CNN
 F 1 "GND" H 2350 4250 50  0000 C CNN
 F 2 "" H 2350 4400 50  0001 C CNN
@@
 $EndComp
 $Comp
-L GND #PWR4
+L GND #PWR5
 U 1 1 5B6684BB
 P 2350 5450
-F 0 "#PWR4" H 2350 5200 50  0001 C CNN
+F 0 "#PWR5" H 2350 5200 50  0001 C CNN
 F 1 "GND" H 2350 5300 50  0000 C CNN
 F 2 "" H 2350 5450 50  0001 C CNN
@@
 	3300 5750 3500 5750
 $Comp
-L GND #PWR8
+L GND #PWR10
 U 1 1 5B66C7B9
 P 3500 5750
-F 0 "#PWR8" H 3500 5500 50  0001 C CNN
+F 0 "#PWR10" H 3500 5500 50  0001 C CNN
 F 1 "GND" H 3500 5600 50  0000 C CNN
 F 2 "" H 3500 5750 50  0001 C CNN
@@
 $EndComp
 $Comp
-L +5V #PWR9
+L +5V #PWR11
 U 1 1 5B66C944
 P 3850 5650
-F 0 "#PWR9" H 3850 5500 50  0001 C CNN
+F 0 "#PWR11" H 3850 5500 50  0001 C CNN
 F 1 "+5V" H 3850 5790 50  0000 C CNN
 F 2 "" H 3850 5650 50  0001 C CNN
@@
 Text Label 4850 5500 0    60   ~ 0
 RST
+$Comp
+L R R5
+U 1 1 5B67508A
+P 2350 3750
+F 0 "R5" V 2250 3750 50  0000 C CNN
+F 1 "2K" V 2350 3750 50  0000 C CNN
+F 2 "Resistors_SMD:R_0603" V 2280 3750 50  0001 C CNN
+F 3 "" H 2350 3750 50  0001 C CNN
+	1    2350 3750
+	0    -1   -1   0
+$EndComp
+$Comp
+L LED D4
+U 1 1 5B67536A
+P 2050 3750
+F 0 "D4" H 2050 3850 50  0000 C CNN
+F 1 "LED" H 2050 3650 50  0000 C CNN
+F 2 "LEDs:LED_0805" H 2050 3750 50  0001 C CNN
+F 3 "" H 2050 3750 50  0001 C CNN
+	1    2050 3750
+	1    0    0    -1
+$EndComp
+$Comp
+L GND #PWR1
+U 1 1 5B675495
+P 1750 3750
+F 0 "#PWR1" H 1750 3500 50  0001 C CNN
+F 1 "GND" H 1750 3600 50  0000 C CNN
+F 2 "" H 1750 3750 50  0001 C CNN
+F 3 "" H 1750 3750 50  0001 C CNN
+	1    1750 3750
+	1    0    0    -1
+$EndComp
+Wire Wire Line
+	1900 3750 1750 3750
+Wire Wire Line
+	2900 3650 2900 3850
+$Comp
+L +12V #PWR6
+U 1 1 5B6758AD
+P 2500 3750
+F 0 "#PWR6" H 2500 3600 50  0001 C CNN
+F 1 "+12V" H 2500 3890 50  0000 C CNN
+F 2 "" H 2500 3750 50  0001 C CNN
+F 3 "" H 2500 3750 50  0001 C CNN
+	1    2500 3750
+	1    0    0    -1
+$EndComp
+$Comp
+L C C16
+U 1 1 5B6763FE
+P 9750 3950
+F 0 "C16" H 9600 4050 50  0000 L CNN
+F 1 "10uf" H 9550 3850 50  0000 L CNN
+F 2 "Capacitors_SMD:C_0603" H 9788 3800 50  0001 C CNN
+F 3 "" H 9750 3950 50  0001 C CNN
+	1    9750 3950
+	-1   0    0    1
+$EndComp
+Connection ~ 9750 3800
+Wire Wire Line
+	9750 4100 10050 4100
+Connection ~ 10050 4100
 $EndSCHEMATC

Commit message: 47/10 divider
Parts:
- C1, C11, C13, C14, C15, C16, C2, C3, C4, C5, C7, C8, C9: symbol C -> Device:C
- C10, C12, C6: symbol CP -> Device:CP
- D1, D2, D3: symbol D_Schottky -> Device:D_Schottky
- D4: symbol LED -> Device:LED
- J1, J2, J4: symbol Conn_01x02 -> UniDCBuckHW-rescue:Conn_01x02
- J3: symbol Conn_01x03 -> UniDCBuckHW-rescue:Conn_01x03
- J5: symbol Conn_01x06_Male -> UniDCBuckHW-rescue:Conn_01x06_Male
- L1: symbol L_Core_Iron -> Device:L_Core_Iron
- Q1: symbol Q_NMOS_GDS -> Device:Q_NMOS_GDS
- R1, R2, R3, R4, R5: symbol R -> Device:R
- U1: symbol LM7812_TO220 -> UniDCBuckHW-rescue:LM7812_TO220
- U2: symbol MCP1703A-5002_SOT23 -> UniDCBuckHW-rescue:MCP1703A-5002_SOT23
- U3: symbol IR2106 -> UniDCBuckHW-rescue:IR2106
- U4: symbol ATTINY85-20SU -> UniDCBuckHW-rescue:ATTINY85-20SU
- U5: symbol ACS712ELCTR-05B-T -> UniDCBuckHW-rescue:ACS712ELCTR-05B-T
